File: tpm2-rgb-stm32/tpm2-rgb-stm32.kicad_sch (KiCad schematic)
At the start: 58 parts

Commit message: added part annotations
Parts:
- gave numbers to parts that had none: 58
Connections:
- net +12V: now also U5.6 (VDD)
- net GATE1: now also U5.7 (NOUTA)
- net GATE2: now also U5.5 (NOUTB)
- net GND: now also R9.2
Other:
- moved on the sheet: U5
