File: tpm2-rgb-stm32/tpm2-rgb-stm32.kicad_sch (KiCad schematic)
At the start: 58 parts, among them J1 Screw_Terminal_01x04, J2 Screw_Terminal_01x08, J3 Screw_Terminal_01x02, J4 Screw_Terminal_01x02, J5 12401832E402A, SW1 SW_Push, U1 COS4426SR, U10 IRF7458TRPBF, U11 IRF7458TRPBF, U12 COS4426SR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

Commit message: touch ups
Connections:
- net SWDCLK: now also U4.37 (PA14)
- net SWDIO: now also U4.34 (PA13)
- no-connect marks 0 -> 48
Other:
- moved on the sheet: C1, C10, C11, C14, C15, C16, C17, C18, C19, C2, C22, C23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
