File: tpm2-rgb-stm32.kicad_pcb (KiCad board)
At the start: 4 copper layers, 1 x 0.7 mm, 59 parts, among them J1 Screw_Terminal_01x04, J2 Screw_Terminal_01x04, J3 Screw_Terminal_01x02, J4 Screw_Terminal_01x02, J5 12401832E402A, J6 Screw_Terminal_01x04, SW1 SW_Push, U1 COS4426SR, U10 IRF7458TRPBF, U11 IRF7458TRPBF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

Commit message: Start layout
Parts:
- J1: value Screw_Terminal_01x04 -> Conn_01x04_Male; footprint TerminalBlock:TerminalBlock_bornier-4_P5.08mm -> Connector_PinHeader_2.54mm:PinHeader_1x04_P2.54mm_Vertical
- moved R3 91.7 mm to (34.1, 9.88), turned to -90 degrees
- moved R4 90.1 mm to (33.8, 16.0), turned to -90 degrees
- moved R9 88.3 mm to (24.9, 97.8)
- moved R11 86.2 mm to (25.0, 106.1)
- moved U2 84.9 mm to (27.9, 9.63), turned to 180 degrees
- moved C13 81.5 mm to (38.5, 21.4)
- moved U13 80.4 mm to (28.1, 47.0), turned to 180 degrees
- moved R6 79.0 mm to (34.1, 28.3), turned to -90 degrees
- moved C3 78.1 mm to (38.4, 18.3)
- moved C4 77.5 mm to (38.6, 10.6)
- moved R5 77.2 mm to (34.1, 22.0), turned to -90 degrees
- moved R12 76.6 mm to (34.1, 46.9), turned to -90 degrees
- moved U1 75.3 mm to (40.5, 14.5), turned to 180 degrees
- moved U6 74.1 mm to (27.9, 22.1), turned to 180 degrees
- moved U3 74.0 mm to (27.7, 15.7), turned to 180 degrees
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Connections:
- J1 pad 1: +5V -> GND
- J1 pad 2: SWDIO -> SWDCLK
- J1 pad 3: SWDCLK -> SWDIO
- J1 pad 4: GND -> +5V
Routing:
- net OUT1: track 0.00 -> 16.6 mm
- net OUT8: track 0.00 -> 12.3 mm
- net OUT2: track 0.00 -> 11.5 mm
- net OUT3: track 0.00 -> 11.1 mm
- net OUT5: track 0.00 -> 10.6 mm
- net OUT4: track 0.00 -> 10.6 mm
- net OUT7: track 0.00 -> 10.4 mm
- net OUT6: track 0.00 -> 10.2 mm
- net GATE6: track 0.00 -> 9.84 mm, vias 0 -> 2
- net GATE4: track 0.00 -> 9.43 mm, vias 0 -> 2
- net GATE2: track 0.00 -> 8.37 mm, vias 0 -> 2
- net GATE5: track 0.00 -> 6.31 mm
- net GATE1: track 0.00 -> 6.10 mm
- net GATE3: track 0.00 -> 5.42 mm
- net Net-(R3-Pad1): track 0.00 -> 4.06 mm
Other:
- board size 1 x 0.7 mm -> 127 x 125.3 mm

Commit message: More PCB layout
Parts:
- moved C10 48.3 mm to (125.3, 60.1)
- moved C21 48.3 mm to (119.8, 61.9)
- moved R10 48.3 mm to (120.0, 72.5)
- moved R2 48.3 mm to (124.7, 66.1)
- moved C20 47.3 mm to (106.3, 84.7)
- moved C6 41.9 mm to (57.1, 57.1)
- moved C8 36.0 mm to (73.4, 54.2), turned to 90 degrees
- moved C5 33.2 mm to (72.0, 50.7), turned to 180 degrees
- moved C9 29.0 mm to (76.2, 57.1)
- moved C7 17.4 mm to (69.8, 63.5), turned to 90 degrees
- moved C15 12.6 mm to (21.8, 90.4)
- moved C14 12.6 mm to (19.8, 90.4)
- moved U9 11.0 mm to (27.5, 90.2)
- moved C16 10.9 mm to (34.4, 87.6)
- moved R1 8.80 mm to (52.7, 94.0), turned to 180 degrees
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Routing:
- net +5V: track 0.00 -> 45.9 mm, vias 0 -> 4
- net +12V: track 0.00 -> 42.8 mm
- net GATE8: track 0.00 -> 15.7 mm, vias 0 -> 4
- net Net-(J5-PadB5): track 0.00 -> 7.08 mm
- net GATE2: track 8.37 -> 13.9 mm, vias 2 -> 4
- net GATE7: track 0.00 -> 5.46 mm
- net GATE4: track 9.43 -> 14.8 mm, vias 2 -> 4
- net +3V3: track 0.00 -> 4.19 mm
- net Net-(R8-Pad1): track 0.00 -> 4.12 mm
- net Net-(R13-Pad1): track 0.00 -> 4.07 mm
- net Net-(R4-Pad1): track 0.00 -> 4.02 mm
- net Net-(R7-Pad1): track 0.00 -> 4.00 mm
- net Net-(R5-Pad1): track 0.00 -> 3.96 mm
- net Net-(R6-Pad1): track 0.00 -> 3.95 mm
- net Net-(R12-Pad1): track 0.00 -> 3.83 mm
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- added copper zone on In1.Cu, net +3V3
- added copper zone on In2.Cu, net +3V3
- added copper zone on B.Cu, net GND
- added copper zone on F.Cu, net GND

Commit message: Do more routing
Parts:
- moved C21 99.6 mm to (34.2, 112.8), turned to -90 degrees
- moved C10 62.7 mm to (63.6, 49.3)
- moved C11 30.2 mm to (70.4, 49.4), turned to 180 degrees
- moved U15 9.18 mm to (27.4, 113.6)
- moved Y1 7.57 mm to (67.2, 45.7)
- moved C5 1.52 mm to (73.4, 51.4)
- moved R11 1.04 mm to (18.6, 108.0)
Connections:
- J5 pad A7: USBDN -> USBDM
- J5 pad B7: USBDN -> USBDM
- U15 pad 15: USDP -> USBDP
- U15 pad 16: USDM -> USBDM
Routing:
- net USBDM: track 0.00 -> 50.0 mm, vias 0 -> 4
- net USBDP: track 0.00 -> 46.7 mm, vias 0 -> 2
- net +5V: track 45.9 -> 67.0 mm, vias 4 -> 6
- net +3V3: track 4.19 -> 23.4 mm, vias 0 -> 7
- net OSC_OUT: track 0.00 -> 9.77 mm
- net OSC_IN: track 0.00 -> 9.13 mm
- net GND: track 0.13 -> 8.38 mm, vias 0 -> 8

Commit message: More work
Parts:
- moved R2 99.1 mm to (31.3, 99.6)
- moved R10 92.2 mm to (33.9, 105.2), turned to 90 degrees
- moved C20 87.6 mm to (26.0, 119.8), turned to 180 degrees
- moved C18 68.3 mm to (35.8, 109.9), turned to 180 degrees
- moved C2 67.6 mm to (53.1, 20.0)
- moved C1 60.0 mm to (60.1, 20.1), turned to 180 degrees
- moved SW1 42.0 mm to (29.4, 63.4), turned to -90 degrees
- moved R1 37.8 mm to (32.8, 62.0), turned to 90 degrees
- moved C9 27.6 mm to (63.5, 32.7), turned to 180 degrees
- moved C8 26.5 mm to (63.3, 29.7), turned to 180 degrees
- moved C7 25.2 mm to (58.2, 41.2), turned to 0 degrees
- moved J3 24.5 mm to (53.5, 6.89)
- moved U4 24.1 mm to (56.4, 33.9)
- moved Y1 24.1 mm to (56.9, 23.9)
- moved C11 24.1 mm to (60.1, 27.6)
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Routing:
- net SWDCLK: track 0.00 -> 94.5 mm, vias 0 -> 8
- net SWDIO: track 0.00 -> 78.0 mm
- net PWM2: track 0.00 -> 49.8 mm
- net +12V: track 42.8 -> 86.9 mm, vias 0 -> 4
- net UART_RX: track 0.00 -> 43.9 mm
- net PWM1: track 0.00 -> 41.9 mm
- net PWM7: track 0.00 -> 21.4 mm
- net PWM8: track 0.00 -> 17.5 mm
- net PWM4: track 0.00 -> 17.4 mm, vias 0 -> 4
- net +3V3: track 23.4 -> 40.0 mm
- net PWM6: track 0.00 -> 15.9 mm, vias 0 -> 4
- net PWM3: track 0.00 -> 11.8 mm
- net PWM5: track 0.00 -> 11.7 mm
- net USBDP: track 46.7 -> 51.1 mm, vias 2 -> 3
- net OSC_IN: track 9.13 -> 13.0 mm
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
Commit message: more routing
Parts:
- moved R10 2.23 mm to (35.7, 106.5), turned to 0 degrees
Routing:
- net Net-(R2-Pad2): track 0.00 -> 85.4 mm, vias 0 -> 4
- net UART_RX: track 43.9 -> 110.2 mm, vias 0 -> 4
- net NRST: track 0.00 -> 55.3 mm, vias 0 -> 4
- net SWDIO: track 78.0 -> 96.6 mm
- net Net-(R10-Pad2): track 0.00 -> 18.5 mm
- net +5V: track 67.0 -> 84.4 mm
- net +3V3: track 40.0 -> 54.1 mm, vias 7 -> 12
- net SWDCLK: track 94.5 -> 92.0 mm

Commit message: Remove swd traces
Routing:
- net SWDIO: track 96.6 -> 0.00 mm
- net SWDCLK: track 92.0 -> 0.00 mm, vias 8 -> 0
- net PWM7: track 21.4 -> 8.61 mm
